Commit message: coboweld replaced cobo_weld

File: src/coboweld_support/urdf/cobo_weld435.xacro (robot description, xacro)
@@ -5,5 +5,5 @@
 -->
 <robot xmlns:xacro="http://ros.org/wiki/xacro"
-       name="cobo_weld" >
+       name="coboweld" >
   <xacro:arg name="transmission_hw_interface" default="hardware_interface/PositionJointInterface"/>
   <!-- ur5 -->
@@ -24,5 +24,5 @@
       <visual>
         <geometry>
-          <mesh filename="package://cobo_weld_support/meshes/collision/STorchRCamKScan.stl"
+          <mesh filename="package://coboweld_support/meshes/collision/STorchRCamKScan.stl"
                 scale="0.001 0.001 0.001"/>
         </geometry>
@@ -31,5 +31,5 @@
       <collision>
         <geometry>
-          <mesh filename="package://cobo_weld_support/meshes/collision/STorchRCamKScan.stl"
+          <mesh filename="package://coboweld_support/meshes/collision/STorchRCamKScan.stl"
                 scale="0.001 0.001 0.001"/>
         </geometry>
