Commit message: Camera and TCP pose adjusted

File: src/coboweld_support/urdf/coboweld435.xacro (robot description, xacro)
@@ -70,5 +70,5 @@
   <xacro:include filename="$(find realsense2_description)/urdf/_d435.urdf.xacro" />
   <xacro:sensor_d435 parent="wrist_3_link" use_nominal_extrinsics="true" name="d435">
-    <origin xyz="0.0 -0.0225 0.18515" rpy="0 ${-pi/2} ${pi/2}"/>
+    <origin xyz="0.0 -0.0225 0.19185" rpy="0 ${-pi/2} ${pi/2}"/>
   </xacro:sensor_d435>
   <link name="table">

Commit message: Almost work

File: src/coboweld_support/urdf/coboweld435.xacro (robot description, xacro)
@@ -70,5 +70,8 @@
   <xacro:include filename="$(find realsense2_description)/urdf/_d435.urdf.xacro" />
   <xacro:sensor_d435 parent="wrist_3_link" use_nominal_extrinsics="true" name="d435">
+    <!--
     <origin xyz="0.0 -0.0225 0.19185" rpy="0 ${-pi/2} ${pi/2}"/>
+    -->
+    <origin xyz="-0.0106 -0.040 0.20435" rpy="0 ${-pi/2} ${pi/2}"/>
   </xacro:sensor_d435>
   <link name="table">

Commit message: The poses of the torch, camera nearly align.

File: src/coboweld_support/urdf/coboweld435.xacro (robot description, xacro)
@@ -42,6 +42,7 @@
     <origin xyz="0.00395 -0.10284 0.37548" rpy="3.1366625 -0.00247520 1.3734586"/>
     <origin xyz="0 -0.111 0.360" rpy="0 0 ${pi}"/>
+    <origin xyz="0.00395 -0.11084 0.36548" rpy="0 0 ${pi}"/>
 -->
-    <origin xyz="0.00395 -0.11084 0.36548" rpy="0 0 ${pi}"/>
+    <origin xyz="0.0 -0.105 0.365" rpy="0 0 ${pi}"/>
     <parent link="wrist_3_link"/>
     <child link="torch"/>
@@ -73,5 +74,5 @@
     <origin xyz="0.0 -0.0225 0.19185" rpy="0 ${-pi/2} ${pi/2}"/>
     -->
-    <origin xyz="-0.0106 -0.040 0.20435" rpy="0 ${-pi/2} ${pi/2}"/>
+    <origin xyz="0.0 -0.0225 0.19185" rpy="0 ${-pi/2} ${pi/2}"/>
   </xacro:sensor_d435>
   <link name="table">

Commit message: So far so good

File: src/coboweld_support/urdf/coboweld435.xacro (robot description, xacro)
@@ -71,8 +71,8 @@
   <xacro:include filename="$(find realsense2_description)/urdf/_d435.urdf.xacro" />
   <xacro:sensor_d435 parent="wrist_3_link" use_nominal_extrinsics="true" name="d435">
+    <origin xyz="0.0 -0.0225 0.19185" rpy="0 ${-pi/2} ${pi/2}"/>
     <!--
-    <origin xyz="0.0 -0.0225 0.19185" rpy="0 ${-pi/2} ${pi/2}"/>
+    <origin xyz="0.003 -0.023 0.19215" rpy="-0.006 -1.570 1.565"/>
     -->
-    <origin xyz="0.0 -0.0225 0.19185" rpy="0 ${-pi/2} ${pi/2}"/>
   </xacro:sensor_d435>
   <link name="table">
